Commit message: tof_array: 新增8个tof传感器

File: src/wheeltec_robot_urdf/wheeltec_robot_urdf/urdf/top_omni_robot.urdf (robot description, URDF)
Before this commit: robot top_omni_robot, 7 links, 6 joints
Links:
- added link tof_link_0; collision cylinder length=0.02 radius=0.01; visual cylinder length=0.02 radius=0.01
- added link tof_link_1; collision cylinder length=0.02 radius=0.01; visual cylinder length=0.02 radius=0.01
- added link tof_link_2; collision cylinder length=0.02 radius=0.01; visual cylinder length=0.02 radius=0.01
- added link tof_link_3; collision cylinder length=0.02 radius=0.01; visual cylinder length=0.02 radius=0.01
- added link tof_link_4; collision cylinder length=0.02 radius=0.01; visual cylinder length=0.02 radius=0.01
- added link tof_link_5; collision cylinder length=0.02 radius=0.01; visual cylinder length=0.02 radius=0.01
- added link tof_link_6; collision cylinder length=0.02 radius=0.01; visual cylinder length=0.02 radius=0.01
- added link tof_link_7; collision cylinder length=0.02 radius=0.01; visual cylinder length=0.02 radius=0.01
Joints:
- added joint tof_joint_0: type fixed, parent base_link, child tof_link_0, origin xyz=0.25 0.0 0.05 rpy=0 0 0
- added joint tof_joint_1: type fixed, parent base_link, child tof_link_1, origin xyz=0.177 -0.177 0.05 rpy=0 0 -0.785
- added joint tof_joint_2: type fixed, parent base_link, child tof_link_2, origin xyz=0.0 -0.25 0.05 rpy=0 0 -1.571
- added joint tof_joint_3: type fixed, parent base_link, child tof_link_3, origin xyz=-0.177 -0.177 0.05 rpy=0 0 -2.356
- added joint tof_joint_4: type fixed, parent base_link, child tof_link_4, origin xyz=-0.25 0.0 0.05 rpy=0 0 3.141
- added joint tof_joint_5: type fixed, parent base_link, child tof_link_5, origin xyz=-0.177 0.177 0.05 rpy=0 0 2.356
- added joint tof_joint_6: type fixed, parent base_link, child tof_link_6, origin xyz=0.0 0.25 0.05 rpy=0 0 1.571
- added joint tof_joint_7: type fixed, parent base_link, child tof_link_7, origin xyz=0.177 0.177 0.05 rpy=0 0 0.785

Commit message: urdf: top_omni: 装了8个tof传感器上去，定义位置完成

File: src/wheeltec_robot_urdf/wheeltec_robot_urdf/urdf/top_omni_robot.urdf (robot description, URDF)
Before this commit: robot top_omni_robot, 15 links, 14 joints
Joints:
- joint tof_joint_0: origin xyz=0.25 0.0 0.05 rpy=0 0 0 -> xyz=0.0 -0.2 0.0 rpy=0 0 -1.57
- joint tof_joint_1: origin xyz=0.177 -0.177 0.05 rpy=0 0 -0.785 -> xyz=0.0516 -0.193 0.0 rpy=0 0 -1.308
- joint tof_joint_2: origin xyz=0.0 -0.25 0.05 rpy=0 0 -1.571 -> xyz=-0.1532 -0.1284 0.0 rpy=0 0 -2.442
- joint tof_joint_3: origin xyz=-0.177 -0.177 0.05 rpy=0 0 -2.356 -> xyz=0.193 -0.0516 0.0 rpy=0 0 -0.262
- joint tof_joint_4: origin xyz=-0.25 0.0 0.05 rpy=0 0 3.141 -> xyz=0.0844 0.1812 0.0 rpy=0 0 1.134
- joint tof_joint_5: origin xyz=-0.177 0.177 0.05 rpy=0 0 2.356 -> xyz=0.193 0.0516 0.0 rpy=0 0 0.262
- joint tof_joint_6: origin xyz=0.0 0.25 0.05 rpy=0 0 1.571 -> xyz=0.0 0.2 0.0 rpy=0 0 -4.710
- joint tof_joint_7: origin xyz=0.177 0.177 0.05 rpy=0 0 0.785 -> xyz=-0.1532 0.1284 0.0 rpy=0 0 -3.838
